Commit message: working on robot model (added cameras)

File: robocluedo_dependencies/robocluedo_hunter_urdf_model/robot/model/robocluedo_urdf.urdf (robot description, URDF)
Before this commit: robot robocluedo_robot, 11 links, 10 joints
Links:
- added link camera_arm
- added link camera_front_low
- added link camera_left
- added link camera_right
Joints:
- added joint joint_camera_arm: type fixed, parent arm_link_03, child camera_arm, origin xyz=0 0 0.1 rpy=0 0 1.57
- added joint joint_camera_front_low: type fixed, parent base_link, child camera_front_low, origin xyz=0.2 0 0.1 rpy=0 0 0
- added joint joint_camera_left: type fixed, parent base_link, child camera_left, origin xyz=0 0.2 0.1 rpy=0 0 1.57
- added joint joint_camera_right: type fixed, parent base_link, child camera_right, origin xyz=0 -0.2 0.1 rpy=0 0 -1.57

File: robocluedo_dependencies/robocluedo_hunter_urdf_model/robot/robocluedo_gazebo_sensing.xacro (robot description, xacro)
@@ -1,35 +1,179 @@
 <?xml version="1.0" ?>
 <robot name="robocluedo_robot" xmlns:xacro="http://www.ros.org/wiki/xacro">
-    <gazebo reference="laser">
-        <sensor name="head_hokuyo_sensor" type="ray">
-            <pose>0 0 0 0 0 0</pose>
-            <visualize>false</visualize>
-            <update_rate>20</update_rate>
-            <ray>
-                <scan>
-                    <horizontal>
-                        <samples>720</samples>
-                        <resolution>1</resolution>
-                        <min_angle>-1.570796</min_angle>
-                        <max_angle>1.570796</max_angle>
-                    </horizontal>
-                </scan>
-                <range>
-                    <min>0.10</min>
-                    <max>10.0</max>
-                    <resolution>0.01</resolution>
-                </range>
-                <noise>
-                    <type>gaussian</type>
-                    <mean>0.0</mean>
-                    <stddev>0.01</stddev>
-                </noise>
-            </ray>
-            <plugin filename="libgazebo_ros_laser.so" name="gazebo_ros_head_hokuyo_controller">
-                <!-- <topicName>m2wr/laser/scan</topicName> -->
-                <topicName>/scan</topicName>
-                <frameName>laser</frameName>
-            </plugin>
-        </sensor>
-    </gazebo>
+	<gazebo reference="laser">
+		<sensor name="head_hokuyo_sensor" type="ray">
+			<pose>0 0 0 0 0 0</pose>
+			<visualize>false</visualize>
+			<update_rate>20</update_rate>
+			<ray>
+				<scan>
+					<horizontal>
+						<samples>720</samples>
+						<resolution>1</resolution>
+						<min_angle>-1.570796</min_angle>
+						<max_angle>1.570796</max_angle>
+					</horizontal>
+				</scan>
+				<range>
+					<min>0.10</min>
+					<max>10.0</max>
+					<resolution>0.01</resolution>
+				</range>
+				<noise>
+					<type>gaussian</type>
+					<mean>0.0</mean>
+					<stddev>0.01</stddev>
+				</noise>
+			</ray>
+			<plugin filename="libgazebo_ros_laser.so" name="gazebo_ros_head_hokuyo_controller">
+				<!-- <topicName>m2wr/laser/scan</topicName> -->
+				<topicName>/scan</topicName>
+				<frameName>laser</frameName>
+			</plugin>
+		</sensor>
+	</gazebo>
+	<gazebo reference="camera_front_low">
+	<sensor type="camera" name="camera_front_low">
+	  <update_rate>30.0</update_rate>
+	  <camera name="camera_front_low">
+		<horizontal_fov>1.3962634</horizontal_fov>
+		<image>
+		  <width>800</width>
+		  <height>800</height>
+		  <format>R8G8B8</format>
+		</image>
+		<clip>
+		  <near>0.02</near>
+		  <far>300</far>
+		</clip>
+		<noise>
+		  <type>gaussian</type>
+		  <mean>0.0</mean>
+		  <stddev>0.007</stddev>
+		</noise>
+	  </camera>
+	  <plugin name="camera_controller" filename="libgazebo_ros_camera.so">
+		<alwaysOn>true</alwaysOn>
+		<updateRate>0.0</updateRate>
+		<cameraName>robocluedo_robot/camera_front_low</cameraName>
+		<imageTopicName>image_raw</imageTopicName>
+		<cameraInfoTopicName>camera_info</cameraInfoTopicName>
+		<frameName>camera_front_low</frameName>
+		<hackBaseline>0.07</hackBaseline>
+		<distortionK1>0.0</distortionK1>
+		<distortionK2>0.0</distortionK2>
+		<distortionK3>0.0</distortionK3>
+		<distortionT1>0.0</distortionT1>
+		<distortionT2>0.0</distortionT2>
+	  </plugin>
+	</sensor>
+	</gazebo>
+	<gazebo reference="camera_left">
+	<sensor type="camera" name="camera_left">
+	  <update_rate>30.0</update_rate>
+	  <camera name="camera_left">
+		<horizontal_fov>1.3962634</horizontal_fov>
+		<image>
+		  <width>800</width>
+		  <height>800</height>
+		  <format>R8G8B8</format>
+		</image>
+		<clip>
+		  <near>0.02</near>
+		  <far>300</far>
+		</clip>
+		<noise>
+		  <type>gaussian</type>
+		  <mean>0.0</mean>
+		  <stddev>0.007</stddev>
+		</noise>
+	  </camera>
+	  <plugin name="camera_controller" filename="libgazebo_ros_camera.so">
+		<alwaysOn>true</alwaysOn>
+		<updateRate>0.0</updateRate>
+		<cameraName>robocluedo_robot/camera_left</cameraName>
+		<imageTopicName>image_raw</imageTopicName>
+		<cameraInfoTopicName>camera_info</cameraInfoTopicName>
+		<frameName>camera_left</frameName>
+		<hackBaseline>0.07</hackBaseline>
+		<distortionK1>0.0</distortionK1>
+		<distortionK2>0.0</distortionK2>
+		<distortionK3>0.0</distortionK3>
+		<distortionT1>0.0</distortionT1>
+		<distortionT2>0.0</distortionT2>
+	  </plugin>
+	</sensor>
+	</gazebo>
+	<gazebo reference="camera_right">
+	<sensor type="camera" name="camera_right">
+	  <update_rate>30.0</update_rate>
+	  <camera name="camera_right">
+		<horizontal_fov>1.3962634</horizontal_fov>
+		<image>
+		  <width>800</width>
+		  <height>800</height>
+		  <format>R8G8B8</format>
+		</image>
+		<clip>
+		  <near>0.02</near>
+		  <far>300</far>
+		</clip>
+		<noise>
+		  <type>gaussian</type>
+		  <mean>0.0</mean>
+		  <stddev>0.007</stddev>
+		</noise>
+	  </camera>
+	  <plugin name="camera_controller" filename="libgazebo_ros_camera.so">
+		<alwaysOn>true</alwaysOn>
+		<updateRate>0.0</updateRate>
+		<cameraName>robocluedo_robot/camera_right</cameraName>
+		<imageTopicName>image_raw</imageTopicName>
+		<cameraInfoTopicName>camera_info</cameraInfoTopicName>
+		<frameName>camera_right</frameName>
+		<hackBaseline>0.07</hackBaseline>
+		<distortionK1>0.0</distortionK1>
+		<distortionK2>0.0</distortionK2>
+		<distortionK3>0.0</distortionK3>
+		<distortionT1>0.0</distortionT1>
+		<distortionT2>0.0</distortionT2>
+	  </plugin>
+	</sensor>
+	</gazebo>
+	<gazebo reference="camera_arm">
+	<sensor type="camera" name="camera_arm">
+	  <update_rate>30.0</update_rate>
+	  <camera name="camera_arm">
+		<horizontal_fov>1.3962634</horizontal_fov>
+		<image>
+		  <width>800</width>
+		  <height>800</height>
+		  <format>R8G8B8</format>
+		</image>
+		<clip>
+		  <near>0.02</near>
+		  <far>300</far>
+		</clip>
+		<noise>
+		  <type>gaussian</type>
+		  <mean>0.0</mean>
+		  <stddev>0.007</stddev>
+		</noise>
+	  </camera>
+	  <plugin name="camera_controller" filename="libgazebo_ros_camera.so">
+		<alwaysOn>true</alwaysOn>
+		<updateRate>0.0</updateRate>
+		<cameraName>robocluedo_robot/camera_arm</cameraName>
+		<imageTopicName>image_raw</imageTopicName>
+		<cameraInfoTopicName>camera_info</cameraInfoTopicName>
+		<frameName>camera_arm</frameName>
+		<hackBaseline>0.07</hackBaseline>
+		<distortionK1>0.0</distortionK1>
+		<distortionK2>0.0</distortionK2>
+		<distortionK3>0.0</distortionK3>
+		<distortionT1>0.0</distortionT1>
+		<distortionT2>0.0</distortionT2>
+	  </plugin>
+	</sensor>
+	</gazebo>
 </robot>

File: robocluedo_dependencies/robocluedo_hunter_urdf_model/robot/robocluedo_sensing.xacro (robot description, xacro)
@@ -1,28 +1,56 @@
 <?xml version="1.0" ?>
 <robot name="robocluedo_robot" xmlns:xacro="http://www.ros.org/wiki/xacro">
-    <link name="laser">
+	<link name="laser">
 		<inertial>
-            <origin rpy="0 0 0" xyz="0 0 0" />
-            <mass value="1" />
-            <inertia ixx="0.0014583333333333334" ixy="0" ixz="0" iyy="0.0014583333333333334" iyz="0" izz="0.0012500000000000002" />
-        </inertial>
-        <visual>
-            <origin rpy="0 0 0" xyz="0 0 0" />
-            <geometry>
-                <cylinder length="0.1" radius="0.05" />
-            </geometry>
-            <material name="white" />
-        </visual>
-        <collision>
-            <origin rpy="0 0 0" xyz="0 0 0" />
-            <geometry>
-                <cylinder length="0.1" radius="0.05" />
-            </geometry>
-        </collision>
-    </link>
-    <joint name="joint_laser" type="fixed">
-        <origin rpy="0 0 0" xyz="0.15 0 0.05" />
-        <parent link="base_link" />
-        <child link="laser" />
-    </joint>
+			<origin rpy="0 0 0" xyz="0 0 0" />
+			<mass value="1" />
+			<inertia ixx="0.0014583333333333334" ixy="0" ixz="0" iyy="0.0014583333333333334" iyz="0" izz="0.0012500000000000002" />
+		</inertial>
+		<visual>
+			<origin rpy="0 0 0" xyz="0 0 0" />
+			<geometry>
+				<cylinder length="0.1" radius="0.05" />
+			</geometry>
+			<material name="white" />
+		</visual>
+		<collision>
+			<origin rpy="0 0 0" xyz="0 0 0" />
+			<geometry>
+				<cylinder length="0.1" radius="0.05" />
+			</geometry>
+		</collision>
+	</link>
+	<joint name="joint_laser" type="fixed">
+		<origin rpy="0 0 0" xyz="0.15 0 0.05" />
+		<parent link="base_link" />
+		<child link="laser" />
+	</joint>
+	<link name="camera_front_low">
+	</link>
+	<joint name="joint_camera_front_low" type="fixed">
+		<origin rpy="0 0 0" xyz="0.2 0 0.1" />
+		<parent link="base_link" />
+		<child link="camera_front_low" />
+	</joint>
+	<link name="camera_left">
+	</link>
+	<joint name="joint_camera_left" type="fixed">
+		<origin rpy="0 0 1.57" xyz="0 0.2 0.1" />
+		<parent link="base_link" />
+		<child link="camera_left" />
+	</joint>
+	<link name="camera_right">
+	</link>
+	<joint name="joint_camera_right" type="fixed">
+		<origin rpy="0 0 -1.57" xyz="0 -0.2 0.1" />
+		<parent link="base_link" />
+		<child link="camera_right" />
+	</joint>
+	<link name="camera_arm">
+	</link>
+	<joint name="joint_camera_arm" type="fixed">
+		<origin rpy="0 0 1.57" xyz="0 0 0.1" />
+		<parent link="arm_link_03" />
+		<child link="camera_arm" />
+	</joint>
 </robot>

Commit message: working on robot model (move_base laser issue)

File: robocluedo_dependencies/robocluedo_hunter_urdf_model/robot/model/robocluedo_urdf.urdf (robot description, URDF)
Before this commit: robot robocluedo_robot, 15 links, 14 joints
Joints:
- joint joint_laser: origin xyz=0.15 0 0.05 rpy=0 0 0 -> xyz=0.2 0 0.05 rpy=0 0 0
- joint joint_left_wheel: origin xyz=0.125 -0.15 0 rpy=0 0 0 -> xyz=0.11 -0.15 0 rpy=0 0 0
- joint joint_right_wheel: origin xyz=0.125 0.15 0 rpy=0 0 0 -> xyz=0.11 0.15 0 rpy=0 0 0

File: robocluedo_dependencies/robocluedo_hunter_urdf_model/robot/robocluedo_chassis.xacro (robot description, xacro)
@@ -87,5 +87,5 @@
     </link>
     <joint name="joint_right_wheel" type="continuous">
-        <origin rpy="0 0 0" xyz="0.125 0.15 0" />
+        <origin rpy="0 0 0" xyz="0.11 0.15 0" />
         <child link="link_right_wheel" />
         <parent link="base_link" />
@@ -95,5 +95,5 @@
     </joint>
     <joint name="joint_left_wheel" type="continuous">
-        <origin rpy="0 0 0" xyz="0.125 -0.15 0" />
+        <origin rpy="0 0 0" xyz="0.11 -0.15 0" />
         <child link="link_left_wheel" />
         <parent link="base_link" />
@@ -113,4 +113,14 @@
                 <cylinder length="0.04" radius="0.1" />
             </geometry>
+            <surface>
+                <friction>
+                    <ode>
+                        <mu>0</mu>
+                        <mu2>0</mu2>
+                        <slip1>1.0</slip1>
+                        <slip2>1.0</slip2>
+                    </ode>
+                </friction>
+            </surface>
         </collision>
         <visual name="link_right_wheel_visual">
@@ -132,4 +142,14 @@
                 <cylinder length="0.04" radius="0.1" />
             </geometry>
+            <surface>
+                <friction>
+                    <ode>
+                        <mu>0</mu>
+                        <mu2>0</mu2>
+                        <slip1>1.0</slip1>
+                        <slip2>1.0</slip2>
+                    </ode>
+                </friction>
+            </surface>
         </collision>
         <visual name="link_left_wheel_visual">

File: robocluedo_dependencies/robocluedo_hunter_urdf_model/robot/robocluedo_gazebo_plugins.xacro (robot description, xacro)
@@ -12,4 +12,5 @@
     </gazebo>
     <gazebo>
+		<!--
         <plugin filename="libgazebo_ros_diff_drive.so" name="differential_drive_controller">
             <legacyMode>true</legacyMode>
@@ -33,4 +34,43 @@
             <publishTf>1</publishTf>
         </plugin>
+        -->
+        <!--
+        <plugin filename="libgazebo_ros_diff_drive.so" name="differential_drive_controller">
+            <legacyMode>true</legacyMode>
+            <alwaysOn>true</alwaysOn>
+            <updateRate>20</updateRate>
+            <leftJoint>joint_right_wheel</leftJoint>
+            <rightJoint>joint_left_wheel</rightJoint>
+            <wheelSeparation>0.3</wheelSeparation>
+            <wheelDiameter>0.2</wheelDiameter>
+            <torque>0.1</torque>
+            <commandTopic>cmd_vel</commandTopic>
+            <odometryTopic>odom</odometryTopic>
+            <odometryFrame>odom</odometryFrame>
+            <robotBaseFrame>base_link</robotBaseFrame>
+            <rosDebugLevel>na</rosDebugLevel>
+            <publishWheelTF>true</publishWheelTF>
+            <publishWheelJointState>true</publishWheelJointState>
+            <wheelAcceleration>0</wheelAcceleration>
+            <wheelTorque>5</wheelTorque>
+            <odometrySource>1</odometrySource>
+            <publishTf>1</publishTf>
+        </plugin>
+        -->
+		<plugin filename="libgazebo_ros_diff_drive.so" name="differential_drive_controller">
+			<legacyMode>true</legacyMode>
+			<alwaysOn>true</alwaysOn>
+			<updateRate>1000</updateRate>
+			<leftJoint>joint_right_wheel</leftJoint>
+			<rightJoint>joint_left_wheel</rightJoint>
+			<wheelSeparation>0.2</wheelSeparation>
+			<wheelDiameter>0.2</wheelDiameter>
+			<torque>0.1</torque>
+			<commandTopic>cmd_vel</commandTopic>
+			<odometryTopic>odom</odometryTopic>
+			<odometryFrame>odom</odometryFrame>
+			<robotBaseFrame>base_link</robotBaseFrame>
+			<odometrySource>world</odometrySource>
+		</plugin>
     </gazebo>
     <gazebo>

File: robocluedo_dependencies/robocluedo_hunter_urdf_model/robot/robocluedo_sensing.xacro (robot description, xacro)
@@ -22,5 +22,5 @@
 	</link>
 	<joint name="joint_laser" type="fixed">
-		<origin rpy="0 0 0" xyz="0.15 0 0.05" />
+		<origin rpy="0 0 0" xyz="0.2 0 0.05" />
 		<parent link="base_link" />
 		<child link="laser" />
